File: hardware/t85.sch (KiCad schematic (older format))
At the start: 4 parts, among them J1 AVRISP6, U1 ATTINY85

Commit message: add documentation + warnings
Other:
- note added: "Warning: This is not isolated and is unsafe.\nIsolate your ethernet sources."
Changed lines of the file:
@@
 Sheet 1 1
 Title ""
-Date "2 sep 2014"
+Date "5 sep 2014"
 Rev ""
 Comp ""
@@
 	6600 2000 6600 2100
 Connection ~ 6600 2050
+Text Notes 1200 3450 0    177  ~ 0
+Warning: This is not isolated and is unsafe.\nIsolate your ethernet sources.
 $EndSCHEMATC
